File: Electronics/electronics.brd (EAGLE design)
At the start: 100 x 80 mm, 0 parts

Commit message: Finished Schematic
Parts:
- added A, B, START: MOMENTARY-SWITCH-SPST-PTH-6.0MM, SparkFun-Switches:TACTILE_SWITCH_PTH_6.0MM
- added A1: LCD, lcd:LCD
- added C1, C14: 0.1uF, SparkFun-Capacitors:0805
- added C10, C11, C13, C2, C3, C4, C5, C6, C7, C8, C9: 1.0uF, SparkFun-Capacitors:0805
- added C12: 10uF, SparkFun-Capacitors:0805
- added C15, C16, C17, C18: 100nF, SparkFun-Capacitors:0805
- added D1: DIFFUSE, SparkFun-LED:LED-RGB-THRU
- added J1: POWER_JACKSLT, SparkFun-Connectors:POWER_JACK_SLOT
- added J2: 455-1750-1-ND, SparkFun-Connectors:1X03
- added LS1: BUZZER-PTH, SparkFun-Electromechanical:BUZZER-12MM
- added MCU: ATMEGA1284P-PU, ATMEGA1284P-PU:DIP254P1524X483-40
- added POWER: (no value), SparkFun-LED:LED_5MM
- added PROG: AVR_SPI_PROG_3X2PTH, SparkFun-Connectors:2X3
- added R1: 200, SparkFun-Resistors:AXIAL-0.3
- added R10, R8, R9: 1k, SparkFun-Resistors:0805
- added R11: 270, SparkFun-Resistors:AXIAL-0.3
- added R12: 10, SparkFun-Resistors:AXIAL-0.3
- added R13, R15, R16, R17, R2: 10k, SparkFun-Resistors:0805
- added R3, R4, R5, R7: 470, SparkFun-Resistors:0805
- added R6: 5k, SparkFun-Resistors:0805
- added S1: (no value), SparkFun-Switches:SWITCH_SPDT_PTH_11.6X4.0MM
- added U$1: JOYSTICK, joystick:JOY
- added U1: V_REG_317SINK, SparkFun-IC-Power:TO220-ADJ
- added VR1: 1k, SparkFun-Resistors:TRIMPOT-PTH-3386U
Connections:
- new net A_X: MCU.35, U$1.A1_2
- new net A_Y: MCU.34, U$1.A2_2
- new net B_A: A.1, C18.2, MCU.39, R17.2
- new net B_B: B.1, C16.2, MCU.38, R15.2
- new net B_SELECT: C15.2, MCU.36, R13.2, U$1.SW2@1, U$1.SW2@2
- new net B_START: C17.2, MCU.37, R16.2, START.1
- new net CS: A1.1, MCU.5, R10.1
- new net GND: A1.15, A1.K, C1.1, C10.2, C11.1, C12.1, C13.1, C14.1, C15.1, C16.1, C17.1, C18.1, C2.2, C3.2, C4.2, C5.2, C6.2, J1.GND@1, J1.GND@2, J2.3, LS1.-, MCU.11, MCU.31, PROG.6, R12.P$1, R13.1, R15.1, R16.1, R17.1, R7.1, R8.1, U$1.A1_3, U$1.A2_3, U$1.SH@1, U$1.SH@2, U$1.SH@3, U$1.SH@4
- new net LCD_A0: A1.3, MCU.1
- new net LCD_C86: A1.27, MCU.2
- new net LCD_E/RD: A1.5, MCU.3
- new net LCD_RW: A1.4, MCU.4
- new net MISO: MCU.7, PROG.1
- new net MOSI: A1.13, MCU.6, PROG.4
- new net N$1: A1.A, VR1.1
- new net N$10: A1.25, C3.1
- new net N$11: A1.24, C4.1
- new net N$12: A1.23, C5.1
- new net N$13: A1.22, C6.1
- new net N$14: A1.19, C8.1
- new net N$15: A1.17, C7.1
- new net N$16: A1.18, C7.2, C8.2
- new net N$17: A1.20, C9.1
- new net N$18: A1.21, C9.2
- new net N$19: A1.16, C10.1
- new net N$2: MCU.19, R3.2
- new net N$20: A1.28, R8.2
- new net N$21: A1.2, R9.2
- new net N$22: MCU.21, R5.2
- new net N$23: LS1.+, MCU.18
- new net N$24: R11.P$1, R12.P$2
- new net N$25: J2.1, MCU.14
- new net N$26: J2.2, MCU.15
- new net N$27: C12.2, S1.2, U1.IN
- new net N$28: R1.P$1, R11.P$2, U1.ADJ
- new net N$3: D1.4, R4.1
- new net N$4: D1.3, R3.1
- new net N$5: D1.1, R5.1
- new net N$6: R6.2, VR1.3
- new net N$7: MCU.20, R4.2
- new net N$8: POWER.K, R7.2
- new net N$9: A1.26, C2.1
- new net RESET: MCU.9, PROG.5, R2.2
- new net SCK: A1.12, MCU.8, PROG.3
- new net VCC: A.3, A1.14, B.3, C1.2, C11.2, C13.2, C14.2, D1.2, MCU.10, MCU.30, POWER.A, PROG.2, R1.P$2, R10.2, R2.1, R6.1, R9.1, START.3, U$1.A1_1, U$1.A2_1, U$1.SW1@1, U$1.SW1@2, U1.OUT
- new net V_BATT: J1.PWR, S1.1

Commit message: Finished PCB routing
Parts:
- removed C15, C16, C17, C18: 100nF, SparkFun-Capacitors:0805
- removed D1: DIFFUSE, SparkFun-LED:LED-RGB-THRU
- removed J1: POWER_JACKSLT, SparkFun-Connectors:POWER_JACK_SLOT
- removed R13, R15, R16, R17: 10k, SparkFun-Resistors:0805
- added LED1: RGB_LED, Keshav Standard:5MM_LED
- added X1: 332-02, con-garry:332-02
- C12: device SparkFun-Capacitors:0805 -> rcl:C1206
- moved C12 484.9 mm to (91.9, 63.1), flipped to the bottom
- moved A 480.8 mm to (72.5, 14.5)
- moved C14 475.7 mm to (53.8, 67.8), flipped to the bottom, turned to 270 degrees
- moved C13 472.8 mm to (56.5, 67.8), flipped to the bottom, turned to 270 degrees
- moved R12 457.8 mm to (95.8, 45.2), turned to 90 degrees
- moved R11 440.9 mm to (92.8, 45.1), turned to 270 degrees
- moved START 437.2 mm to (50.0, 5.00)
- moved R1 423.5 mm to (88.8, 45.1), turned to 270 degrees
- moved R10 382.3 mm to (68.2, 63.8), flipped to the bottom, turned to 90 degrees
- moved R9 378.8 mm to (66.0, 63.8), flipped to the bottom, turned to 270 degrees
- moved C10 369.7 mm to (50.2, 67.8), flipped to the bottom, turned to 90 degrees
- moved R7 366.5 mm to (96.5, 56.5), flipped to the bottom, turned to 180 degrees
- moved C1 365.3 mm to (50.0, 50.5), flipped to the bottom, turned to 180 degrees
- moved C9 363.5 mm to (41.5, 67.8), flipped to the bottom, turned to 270 degrees
- moved C8 363.3 mm to (45.0, 67.8), flipped to the bottom, turned to 90 degrees
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Connections:
- net A_X: now also MCU.36; no longer MCU.35
- net A_Y: now also MCU.35; no longer MCU.34
- net B_A: now also MCU.38; no longer C18.2, MCU.39, R17.2
- net B_B: now also MCU.39; no longer C16.2, MCU.38, R15.2
- net B_SELECT: now also MCU.34, U$1.SW1@1, U$1.SW1@2; no longer C15.2, MCU.36, R13.2, U$1.SW2@1, U$1.SW2@2
- net B_START: no longer C17.2, R16.2
- net GND: now also A.3, B.3, C12.2, J2.1, START.3, U$1.SW2@1, U$1.SW2@2, X1.2; no longer C12.1, C15.1, C16.1, C17.1, C18.1, J1.GND@1, J1.GND@2, J2.3, R13.1, R15.1, R16.1, R17.1
- net LCD_A0: no longer MCU.1
- net LCD_C86: no longer MCU.2
- net LCD_E/RD: no longer MCU.3
- net LCD_RW: no longer MCU.4
- net N$1: now also VR1.2
- net N$25: now also J2.2; no longer J2.1
- net N$26: now also J2.3; no longer J2.2
- net N$27: now also C12.1; no longer C12.2
- net N$3: now also LED1.G; no longer D1.4
- net N$4: now also LED1.R; no longer D1.3
- net N$5: now also LED1.B; no longer D1.1
- net VCC: now also LED1.C; no longer A.3, B.3, D1.2, START.3, U$1.SW1@1, U$1.SW1@2
- net V_BATT: now also X1.1; no longer J1.PWR
Routing:
- net VCC: track 0.00 -> 294.6 mm
- net A_Y: track 0.00 -> 73.2 mm
- net B_SELECT: track 0.00 -> 64.9 mm
- net A_X: track 0.00 -> 59.8 mm
- net MOSI: track 0.00 -> 54.0 mm, vias 0 -> 1
- net B_START: track 0.00 -> 50.9 mm
- net SCK: track 0.00 -> 43.4 mm
- net RESET: track 0.00 -> 42.9 mm
- net N$5: track 0.00 -> 30.9 mm
- net N$28: track 0.00 -> 30.0 mm
- net MISO: track 0.00 -> 29.2 mm
- net N$25: track 0.00 -> 27.9 mm
- net N$23: track 0.00 -> 26.5 mm
- net N$26: track 0.00 -> 22.9 mm
- net B_B: track 0.00 -> 22.8 mm
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- added copper zone on layer 16, net GND
Other:
- board size 100 x 80 mm -> 100 x 70 mm
