File: Electronics/electronics.sch (EAGLE design)
At the start: 0 parts

Commit message: Finished Schematic
Parts:
- added A, B, START: MOMENTARY-SWITCH-SPST-PTH-6.0MM, SparkFun-Switches:MOMENTARY-SWITCH-SPST-PTH-6.0MM
- added A1: LCD, lcd:LCD
- added C1, C14: 0.1uF, SparkFun-Capacitors:1.0UF-0805-25V-10%
- added C10, C11, C13, C2, C3, C4, C5, C6, C7, C8, C9: 1.0uF, SparkFun-Capacitors:1.0UF-0805-25V-10%
- added C12: 10uF, SparkFun-Capacitors:1.0UF-0805-25V-10%
- added C15, C16, C17, C18: 100nF, SparkFun-Capacitors:1.0UF-0805-25V-10%
- added D1: DIFFUSE, SparkFun-LED:LED-RGB-CADIFFUSE
- added J1: POWER_JACKSLT, SparkFun-Connectors:POWER_JACKSLT
- added J2: 455-1750-1-ND, SparkFun-Connectors:CONN_03
- added LS1: BUZZER-PTH, SparkFun-Electromechanical:BUZZER-PTH
- added MCU: ATMEGA1284P-PU, ATMEGA1284P-PU:ATMEGA1284P-PU
- added POWER: (no value), SparkFun-LED:LED5MM
- added PROG: AVR_SPI_PROG_3X2PTH, SparkFun-Connectors:AVR_SPI_PROG_3X2PTH
- added R1: 200, SparkFun-Resistors:1KOHM-HORIZ-1/4W-1%
- added R10, R8, R9: 1k, SparkFun-Resistors:0.3OHM-0805-1/8W-1%
- added R11: 270, SparkFun-Resistors:1KOHM-HORIZ-1/4W-1%
- added R12: 10, SparkFun-Resistors:1KOHM-HORIZ-1/4W-1%
- added R13, R15, R16, R17, R2: 10k, SparkFun-Resistors:0.3OHM-0805-1/8W-1%
- added R3, R4, R5, R7: 470, SparkFun-Resistors:0.3OHM-0805-1/8W-1%
- added R6: 5k, SparkFun-Resistors:0.3OHM-0805-1/8W-1%
- added S1: (no value), SparkFun-Switches:SWITCH-SPDT-PTH-11.6X4.0MM
- added U$1: JOYSTICK, joystick:JOYSTICK
- added U1: V_REG_317SINK, SparkFun-IC-Power:V_REG_317SINK
- added VR1: 1k, SparkFun-Resistors:TRIMPOT-PTH-10MM-KNOB-1/2W-10%
Connections:
- new net A_X: MCU.PA5, U$1.A1_2
- new net A_Y: MCU.PA6, U$1.A2_2
- new net B_A: A.1, C18.2, MCU.PA1, R17.2
- new net B_B: B.1, C16.2, MCU.PA2, R15.2
- new net B_SELECT: C15.2, MCU.PA4, R13.2, U$1.SW2@1, U$1.SW2@2
- new net B_START: C17.2, MCU.PA3, R16.2, START.1
- new net CS: A1.!CS1, MCU.PB4, R10.1
- new net GND: A1.K, A1.VSS, C1.1, C10.2, C11.1, C12.1, C13.1, C14.1, C15.1, C16.1, C17.1, C18.1, C2.2, C3.2, C4.2, C5.2, C6.2, J1.GND, J1.GNDBREAK, J2.3, LS1.2, MCU.GND, MCU.GND_2, PROG.6, R12.1, R13.1, R15.1, R16.1, R17.1, R7.1, R8.1, U$1.A1_3, U$1.A2_3, U$1.SH@1, U$1.SH@2, U$1.SH@3, U$1.SH@4
- new net LCD_A0: A1.A0, MCU.PB0
- new net LCD_C86: A1.C86, MCU.PB1
- new net LCD_E/RD: A1.E/RD, MCU.PB2
- new net LCD_RW: A1.RW/WR, MCU.PB3
- new net MISO: MCU.PB6, PROG.1
- new net MOSI: A1.DB7, MCU.PB5, PROG.4
- new net N$1: A1.A, VR1.CCW
- new net N$10: A1.V1, C3.1
- new net N$11: A1.V2, C4.1
- new net N$12: A1.V3, C5.1
- new net N$13: A1.V4, C6.1
- new net N$14: A1.CAP1P, C8.1
- new net N$15: A1.CAP3P, C7.1
- new net N$16: A1.CAP1N, C7.2, C8.2
- new net N$17: A1.CAP2P, C9.1
- new net N$18: A1.CAP2N, C9.2
- new net N$19: A1.VOUT, C10.1
- new net N$2: MCU.PD5, R3.2
- new net N$20: A1.PS, R8.2
- new net N$21: A1.!RES, R9.2
- new net N$22: MCU.PD7, R5.2
- new net N$23: LS1.1, MCU.PD4
- new net N$24: R11.1, R12.2
- new net N$25: J2.1, MCU.PD0
- new net N$26: J2.2, MCU.PD1
- new net N$27: C12.2, S1.P, U1.IN
- new net N$28: R1.1, R11.2, U1.ADJ
- new net N$3: D1.BLU, R4.1
- new net N$4: D1.GRN, R3.1
- new net N$5: D1.RED, R5.1
- new net N$6: R6.2, VR1.CW
- new net N$7: MCU.PD6, R4.2
- new net N$8: POWER.C, R7.2
- new net N$9: A1.V0, C2.1
- new net RESET: MCU.~RESET, PROG.5, R2.2
- new net SCK: A1.DB6, MCU.PB7, PROG.3
- new net VCC: A.2, A1.VDD, B.2, C1.2, C11.2, C13.2, C14.2, D1.A, MCU.AVCC, MCU.VCC, POWER.A, PROG.2, R1.2, R10.2, R2.1, R6.1, R9.1, START.2, U$1.A1_1, U$1.A2_1, U$1.SW1@1, U$1.SW1@2, U1.OUT
- new net V_BATT: J1.PWR, S1.O

Commit message: Finished PCB routing
Parts:
- removed C15, C16, C17, C18: 100nF, SparkFun-Capacitors:1.0UF-0805-25V-10%
- removed D1: DIFFUSE, SparkFun-LED:LED-RGB-CADIFFUSE
- removed J1: POWER_JACKSLT, SparkFun-Connectors:POWER_JACKSLT
- removed R13, R15, R16, R17: 10k, SparkFun-Resistors:0.3OHM-0805-1/8W-1%
- added LED1: RGB_LED, Keshav Standard:RGB_LED
- added X1: 332-02, con-garry:332-02
- C12: device SparkFun-Capacitors:1.0UF-0805-25V-10% -> rcl:C-USC1206
Connections:
- net A_X: now also MCU.PA4; no longer MCU.PA5
- net A_Y: now also MCU.PA5; no longer MCU.PA6
- net B_A: now also MCU.PA2; no longer C18.2, MCU.PA1, R17.2
- net B_B: now also MCU.PA1; no longer C16.2, MCU.PA2, R15.2
- net B_SELECT: now also MCU.PA6, U$1.SW1@1, U$1.SW1@2; no longer C15.2, MCU.PA4, R13.2, U$1.SW2@1, U$1.SW2@2
- net B_START: no longer C17.2, R16.2
- net GND: now also A.2, B.2, C12.2, J2.1, START.2, U$1.SW2@1, U$1.SW2@2, X1-2.S; no longer C12.1, C15.1, C16.1, C17.1, C18.1, J1.GND, J1.GNDBREAK, J2.3, R13.1, R15.1, R16.1, R17.1
- net LCD_A0: no longer MCU.PB0
- net LCD_C86: no longer MCU.PB1
- net LCD_E/RD: no longer MCU.PB2
- net LCD_RW: no longer MCU.PB3
- net N$1: now also VR1.WIPER
- net N$25: now also J2.2; no longer J2.1
- net N$26: now also J2.3; no longer J2.2
- net N$27: now also C12.1; no longer C12.2
- net N$3: now also LED1.G; no longer D1.BLU
- net N$4: now also LED1.R; no longer D1.GRN
- net N$5: now also LED1.B; no longer D1.RED
- net VCC: now also LED1.A; no longer A.2, B.2, D1.A, START.2, U$1.SW1@1, U$1.SW1@2
- net V_BATT: now also X1-1.S; no longer J1.PWR
Other:
- moved on the sheet: C12, J2
